File: Mini EVSE.sch (KiCad schematic (older format))
At the start: 33 parts, among them IC1 G3MC-201PL DC5, IC2 IRM-03-5, IC3 ATTINY84-20PU, IC4 TMR1-0522, IC5 SI8261BAC-C-IP, J1 RE OUT, J10 M, J2 AC IN, J4 ICP, J5 SWITCH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

Commit message: Update to Kicad 5
Parts:
- C1, C2, C3, C4, C5: symbol C_Small -> Device:C_Small
- D1: symbol D_TVS -> Device:D_TVS
- D2: symbol D_Zener -> Device:D_Zener
- F1: symbol Fuse -> Device:Fuse
- IC1: symbol S102S01 -> Relay_SolidState:S102S01
- IC2: symbol IRM-03-5 -> Converter_ACDC:IRM-03-5
- IC3: symbol ATTINY84-20PU -> MCU_Microchip_ATtiny:ATtiny84-20PU
- IC4: symbol TMR1-0522 -> miscellaneous:TMR1-0522
- IC5: symbol SI8261BAC-C-IP -> miscellaneous:SI8261BAC-C-IP
- J1, J2: symbol CONN_01X02_MALE -> Connector:Conn_01x02_Male
- J10, J7, J8, J9: symbol CONN_01X01_FEMALE -> Mechanical:MountingHole_Pad
- J4, J5: symbol CONN_02X03 -> Connector_Generic:Conn_02x03_Odd_Even
- J6: symbol CONN_01X03_MALE -> Connector:Conn_01x03_Male
- R1, R10, R2, R3, R4, R5, R6, R7, R8, R9: symbol R -> Device:R
- X1: symbol Crystal_Small -> Device:Crystal_Small
Connections:
- wire segments 99 -> 117
